Commit message: commit to update

File: urdf/mybot.xacro (robot description, xacro)
@@ -69,4 +69,7 @@
     </collision>
   </link>
+  <gazebo reference="base_link">
+    <material>Gazebo/Orange</material>
+  </gazebo>
   <!--base_link to base_footprint Joint-->
   <joint name="base_link_joint" type="fixed">
@@ -92,4 +95,7 @@
     <xacro:sphere_inertia m="${caster_wheel_mass}" r="${caster_wheel_radius}"/>
   </link>
+  <gazebo reference="caster_wheel">
+    <material>Gazebo/Blue</material>
+  </gazebo>
   <!--Caster Wheel Joint-->
   <joint name="caster_wheel_joint" type="continuous">
@@ -117,4 +123,7 @@
       <xacro:cylinder_inertia m="${wheel_mass}" r="${wheel_radius}" h="0.005"/>
     </link>
+  <gazebo reference="${prefix}_wheel">
+    <material>Gazebo/Blue</material>
+  </gazebo>
     <joint name="${prefix}_wheel_joint" type="continuous">
       <axis xyz="-0.06 1 0" rpy="0 0 0" />
@@ -127,3 +136,4 @@
   <xacro:wheel prefix="left_back" reflect="1"/>
   <xacro:wheel prefix="right_back" reflect="-1"/>
+  <xacro:include filename="$(find my_bot)/urdf/mybot_gazebo_plugins.xacro"/>
 </robot>

Commit message: commit for update

File: urdf/mybot.xacro (robot description, xacro)
@@ -11,4 +11,5 @@
   <xacro:property name="wheel_mass" value="1"/>
   <xacro:property name="base_mass" value="5"/>
+  <xacro:include filename="$(find my_bot)/urdf/mybot_gazebo_plugins.xacro"/>
   <!--Color Properties-->
   <material name="blue">
@@ -136,4 +137,25 @@
   <xacro:wheel prefix="left_back" reflect="1"/>
   <xacro:wheel prefix="right_back" reflect="-1"/>
-  <xacro:include filename="$(find my_bot)/urdf/mybot_gazebo_plugins.xacro"/>
+  <!-- Hokuyo Laser -->
+  <link name="hokuyo_laser">
+    <visual>
+      <origin xyz="0.01 0 0.043" rpy="0 0 0"/>
+      <geometry>
+        <mesh filename="package://my_bot/meshes/hokuyo.dae"/>
+      </geometry>
+    </visual>
+    <collision>
+      <origin xyz="0 0 0" rpy="0 0 0"/>
+      <geometry>
+        <box size="0.05 0.05 0.05"/>
+      </geometry>
+    </collision>
+    <xacro:box_inertia m="0.2" w="0.05" h="0.05" d="0.05"/>
+  </link>
+  <joint name="hokuyo_joint" type="fixed">
+    <axis xyz="0 1 0" />
+    <origin xyz="0.01 0 0.043" rpy="0 0 0"/>
+    <parent link="base_link"/>
+    <child link="hokuyo_laser"/>
+  </joint>
 </robot>

File: urdf/mybot_gazebo_plugins.xacro (robot description, xacro)
@@ -17,3 +17,35 @@
     </plugin>
   </gazebo>
+  <!--Gazebo Hokuyo Laser Plugin-->
+  <gazebo reference="hokuyo_laser">
+    <sensor type="gpu_ray" name="head_hokuyo_sensor">
+      <pose>0 0 0 0 0 0</pose>
+      <visualize>true</visualize>
+      <update_rate>20</update_rate>
+      <ray>
+        <scan>
+          <horizontal>
+            <samples>1440</samples>
+            <resolution>1</resolution>
+            <min_angle>-3.14159</min_angle>
+            <max_angle>3.14159</max_angle>
+          </horizontal>
+        </scan>
+        <range>
+          <min>0.10</min>
+          <max>30.0</max>
+          <resolution>0.01</resolution>
+        </range>
+        <noise>
+          <type>gaussian</type>
+          <mean>0.0</mean>
+          <stddev>0.01</stddev>
+        </noise>
+      </ray>
+      <plugin name="gazebo_ros_head_hokuyo_controller" filename="libgazebo_ros_laser.so">
+        <topicName>/mybot/laser_scan/scan</topicName>
+        <frameName>hokuyo_laser</frameName>
+      </plugin>
+    </sensor>
+  </gazebo>
 </robot>
